Commit message: new urdf added

File: ros_ws/src/robot_description/urdf/robot_description.urdf (robot description, URDF)
Before this commit: robot rover.SLDASM, 4 links, 3 joints
Links:
- link base_link: geometry collision mesh filename=package://robot_description/meshes/base_link.STL; visual mesh filename=package://robot_description/meshes/base_link.STL
- link left_wheel: geometry collision mesh filename=package://robot_description/meshes/left_wheel.STL; visual mesh filename=package://robot_description/meshes/left_wheel.STL
- link lidar: geometry collision mesh filename=package://robot_description/meshes/lidar.STL; visual mesh filename=package://robot_description/meshes/lidar.STL
- link right_wheel: geometry collision mesh filename=package://robot_description/meshes/right_wheel.STL; visual mesh filename=package://robot_description/meshes/right_wheel.STL

Commit message: lidar on pi comming with pc

File: ros_ws/src/robot_description/urdf/robot_description.urdf (robot description, URDF)
Before this commit: robot rover.SLDASM, 4 links, 3 joints
Joints:
- joint lidar_joint: origin xyz=0 0.00508 0.1196 rpy=1.5708 0 0 -> xyz=0 0.00508 0.1196 rpy=0 0 0
